File: electrical/rpi/robot.sch (KiCad schematic (older format))
At the start: 9 parts, among them J1 i2c, J2 Pi Header, J4 i2c, J6 Power/Data Input, Q1 BSS138, U2 74LVC1G125, U3 74LVC1G126

Commit message: new board :electric_plug:  :bento:
Parts:
- added J3: 12V/Data, Connectors_Molex:Molex_SPOX-5267_22-03-5035_03x2.54mm_Straight, symbol robot-rescue:Conn_01x03
- J2: symbol Connector_Generic:Conn_02x05_Odd_Even -> robot-rescue:Conn_02x05_Odd_Even-Connector_Generic
- J6: value Power/Data Input -> 5V/Data
- R2, R3: symbol Device:R -> robot-rescue:R-Device
Connections:
- net DATA: now also J3.1 (Pin_1)
- net GND: now also J3.3 (Pin_3)
- no-connect marks 0 -> 1
Changed lines of the file:
@@
 $EndDescr
 $Comp
-L power:PWR_FLAG #FLG01
+L robot-rescue:PWR_FLAG-power #FLG01
 U 1 1 5A7E28CA
 P 4150 7050
@@
 $EndComp
 $Comp
-L power:GND #PWR02
+L robot-rescue:GND-power #PWR02
 U 1 1 5A7E2968
 P 4150 7150
@@
 Robotis AX-12A Servo Data to Serial Converter
 $Comp
-L power:GND #PWR03
+L robot-rescue:GND-power #PWR03
 U 1 1 5A93AA24
 P 4900 2300
@@
 $EndComp
 $Comp
-L power:+3V3 #PWR07
+L robot-rescue:+3V3-power #PWR07
 U 1 1 5AA1ADF2
 P 3500 1900
@@
 $EndComp
 $Comp
-L Device:R R3
+L robot-rescue:R-Device R3
 U 1 1 5AA2CFAD
 P 7800 4150
@@
 $EndComp
 $Comp
-L Device:R R2
+L robot-rescue:R-Device R2
 U 1 1 5AA2CFFB
 P 8450 4150
@@
 $EndComp
 $Comp
-L power:+5V #PWR09
+L robot-rescue:+5V-power #PWR09
 U 1 1 5AA2D056
 P 8450 3850
@@
 RXI
 $Comp
-L power:+5V #PWR010
+L robot-rescue:+5V-power #PWR010
 U 1 1 5AA2F235
 P 3100 6950
@@
 $EndComp
 $Comp
-L power:PWR_FLAG #FLG011
+L robot-rescue:PWR_FLAG-power #FLG011
 U 1 1 5AA2F273
 P 3100 7150
@@
 DATA
 $Comp
-L power:GND #PWR012
+L robot-rescue:GND-power #PWR012
 U 1 1 5AA31552
 P 6300 2200
@@
 Connection ~ 7800 4400
 $Comp
-L power:+5V #PWR013
+L robot-rescue:+5V-power #PWR013
 U 1 1 5AAD5DA7
 P 4400 1900
@@
 	7800 4750 9000 4750
 $Comp
-L power:+3V3 #PWR014
+L robot-rescue:+3V3-power #PWR014
 U 1 1 5B844AC7
 P 7800 3850
@@
 P 6650 2050
 F 0 "J6" H 6650 2250 50  0000 C CNN
-F 1 "Power/Data Input" H 6750 1800 50  0000 C CNN
+F 1 "5V/Data" H 6650 1800 50  0000 C CNN
 F 2 "Connectors_Molex:Molex_SPOX-5267_22-03-5035_03x2.54mm_Straight" H 6650 2050 50  0001 C CNN
 F 3 "" H 6650 2050 50  0001 C CNN
@@
 	5850 2050 5850 1950
 $Comp
-L power:+5V #PWR018
+L robot-rescue:+5V-power #PWR018
 U 1 1 5B8453C9
 P 5850 1950
@@
 $EndComp
 $Comp
-L power:GND #PWR023
+L robot-rescue:GND-power #PWR023
 U 1 1 5B8896CA
 P 3600 2500
@@
 $EndComp
 $Comp
-L Connector_Generic:Conn_02x05_Odd_Even J2
+L robot-rescue:Conn_02x05_Odd_Even-Connector_Generic J2
 U 1 1 5BFB75E1
 P 3900 2200
@@
 SCL
 $Comp
-L power:GND #PWR0101
+L robot-rescue:GND-power #PWR0101
 U 1 1 5BFC0448
 P 2500 3100
@@
 $EndComp
 $Comp
-L power:+3V3 #PWR0102
+L robot-rescue:+3V3-power #PWR0102
 U 1 1 5BFC049F
 P 2400 1900
@@
 	2350 2300 2250 2300
 $Comp
-L power:VCC #PWR0103
+L robot-rescue:VCC-power #PWR0103
 U 1 1 5BFD7D0B
 P 3450 6950
@@
 $EndComp
 $Comp
-L power:+3V3 #PWR0104
+L robot-rescue:+3V3-power #PWR0104
 U 1 1 5BFD9890
 P 3650 6950
@@
 $EndComp
 $Comp
-L power:PWR_FLAG #FLG0101
+L robot-rescue:PWR_FLAG-power #FLG0101
 U 1 1 5BFD98B4
 P 3650 7150
@@
 Wire Wire Line
 	3650 7050 3650 6950
+$Comp
+L robot-rescue:Conn_01x03 J3
+U 1 1 5BFDAA78
+P 6650 1350
+F 0 "J3" H 6650 1550 50  0000 C CNN
+F 1 "12V/Data" H 6650 1100 50  0000 C CNN
+F 2 "Connectors_Molex:Molex_SPOX-5267_22-03-5035_03x2.54mm_Straight" H 6650 1350 50  0001 C CNN
+F 3 "" H 6650 1350 50  0001 C CNN
+	1    6650 1350
+	1    0    0    -1
+$EndComp
+$Comp
+L robot-rescue:GND-power #PWR0105
+U 1 1 5BFDAB28
+P 6300 1550
+F 0 "#PWR0105" H 6300 1300 50  0001 C CNN
+F 1 "GND" H 6300 1400 50  0000 C CNN
+F 2 "" H 6300 1550 50  0001 C CNN
+F 3 "" H 6300 1550 50  0001 C CNN
+	1    6300 1550
+	1    0    0    -1
+$EndComp
+Text GLabel 6300 1250 0    60   BiDi ~ 0
+DATA
+NoConn ~ 6450 1350
+Wire Wire Line
+	6450 1450 6300 1450
+Wire Wire Line
+	6300 1450 6300 1550
+Wire Wire Line
+	6450 1250 6300 1250
 $EndSCHEMATC
