File: electrical/power-v6/robot.kicad_pcb (KiCad board)
At the start: 2 copper layers, 49.5 x 49.5 mm, 20 parts, among them J1 C1-2, J10 LEG2, J11 EXT, J12 LEG4, J13 EXT, J14 C3-4, J15 LEG3, J2 RPi, J3 Data, J4 Leg1-2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

Commit message: new board :electric_plug:  :bento:
Parts:
- added J16: 5V, Pin_Headers:Pin_Header_Straight_1x02_Pitch2.54mm, F.Cu at (117.5, 103.5)
- added J17: 12V, Pin_Headers:Pin_Header_Straight_1x02_Pitch2.54mm, F.Cu at (150.5, 103.5)
- added J18: 12V, Pin_Headers:Pin_Header_Straight_1x02_Pitch2.54mm, F.Cu at (146.7, 103.5)
- added J9: 5V, Pin_Headers:Pin_Header_Straight_1x02_Pitch2.54mm, F.Cu at (121.3, 103.5)
- J4, J7: footprint Wire_Connections_Bridges:WireConnection_2.50mmDrill_LargePad -> Wire_Connections_Bridges:WireConnection_1.50mmDrill
- moved R1 37.5 mm to (123.3, 91.4)
- moved D1 37.1 mm to (123.3, 95.9), turned to 180 degrees
- moved J2 5.99 mm to (136.5, 91.4)
- moved J4 4.68 mm to (121.9, 63.5)
- moved J7 3.11 mm to (150.5, 63.5)
- moved J5 1.08 mm to (130.8, 100.3)
- renumbered H1 to ?, H2 to ?, H3 to ?, H4 to ?
Routing:
- net Net-(J12-Pad2): track 0.00 -> 120.8 mm
- net Net-(D1-Pad2): track 56.2 -> 146.9 mm
- net DATA: track 0.00 -> 88.9 mm
- net +5V: track 0.00 -> 35.1 mm
- net Net-(D1-Pad1): track 0.00 -> 7.49 mm
Other:
- board text added: "12V G"
- board text added: "12V GND"
- board text added: "5V G"
- board text added: "D 12 G"
- board text added: "EN 12V GND GND 5V"
- board text added: "GND 12V"
- board text removed: "DAT 12V GND"

Commit message: up
Parts:
- removed ? (x4): MountingHole, Mounting_Holes:MountingHole_2.2mm_M2
- added H1: MountingHole, MountingHole:MountingHole_2.5mm, F.Cu at (111.8, 62.5)
- added H2: MountingHole, MountingHole:MountingHole_2.5mm, F.Cu at (111.8, 106.7)
- added H3: MountingHole, MountingHole:MountingHole_2.5mm, F.Cu at (156.2, 62.5)
- added H4: MountingHole, MountingHole:MountingHole_2.5mm, F.Cu at (156.2, 106.7)
- added LOGO1: Logo_Open_Hardware_Large, Symbol:OSHW-Logo2_24.3x20mm_SilkScreen, B.Cu at (133.3, 78.7)
- J5: footprint Connectors:USB_A -> Connector_USB:USB_A_Wuerth_61400826021_Horizontal_Stacked
Routing:
- net +5V: track 35.1 -> 20.6 mm

Commit message: up
Parts:
- J5: value USB_A -> USB_A_2_PORT
- renumbered H1 to ?, H2 to ?, H3 to ?, H4 to ?
Connections:
- J5 pad 5: GND -> +5V
- J5 pad 8: (no net) -> GND
- J5 pad 9: (no net) -> GND
Routing:
- net +5V: track 20.6 -> 34.8 mm
